File: ATTiny/microprocessor.kicad_sch (KiCad schematic)
At the start: 1 part, among them U1 ATtiny102-M

Commit message: update
Parts:
- removed U1: ATtiny102-M, Package_DFN_QFN:DFN-8-1EP_3x2mm_P0.5mm_EP1.3x1.5mm, symbol MCU_Microchip_ATtiny:ATtiny102-M
- added C5, C6: 22pF, symbol Device:C_Polarized_Small_US
- added U1: ATtiny85-20M, Package_DFN_QFN:QFN-20-1EP_4x4mm_P0.5mm_EP2.6x2.6mm, symbol MCU_Microchip_ATtiny:ATtiny85-20M
- added Y1: 12MHz, symbol Device:Crystal_Small
Connections:
- net GND: now also C5.2, C6.2, U1.21 (GND), U1.8 (GND)
- net VCC: now also U1.15 (VCC)
- new net: C6.1, U1.5 (XTAL2/PB4), Y1.1
- new net: C5.1, U1.2 (XTAL1/PB3), Y1.2
- new net TUNER_OUTPUT: U1.14 (PB2)
- no-connect marks 6 -> 0
