File: Arduino/Finus-ARDUINO.kicad_sch (KiCad schematic)
At the start: 16 parts

Commit message: update
Parts:
- removed R?: 480, symbol Device:R_Small
- gave numbers to parts that had none: 13
Connections:
- net at DS1.15 (LED(+)): now also A1.5 (+5V), C4.2, DS1.2 (VDD), R1.1, RV1.3, U1.8 (V+)
- no-connect marks 0 -> 28
Other:
- title: Finus - Digital Tuner -> Finus
- moved on the sheet: RV1
